File: hardware/boards/GDOv5 Board/GDOv5 Board.brd (EAGLE design)
At the start: 100 x 80 mm, 27 parts, among them IC1 DS1820, IC2 REG1117, J1 DCJ0202

Commit message: Updating routing and layout
Parts:
- removed S1: (no value), adafruit:B3F-40XX
- moved D1 75.7 mm to (21.6, 8.89), turned to 180 degrees
- moved JP1 71.4 mm to (20.3, 5.08), turned to 180 degrees
- moved D3 65.5 mm to (26.7, 14.0), turned to 180 degrees
- moved D2 63.8 mm to (26.7, 8.89), turned to 180 degrees
- moved R4 58.9 mm to (17.8, 26.7), turned to 90 degrees
- moved C6 54.3 mm to (21.6, 20.3), turned to 90 degrees
- moved R5 51.4 mm to (3.81, 61.0), turned to 180 degrees
- moved R6 50.6 mm to (25.4, 26.7), turned to 90 degrees
- moved C7 48.4 mm to (29.2, 20.3), turned to 90 degrees
- moved IC1 47.8 mm to (3.81, 66.0), turned to 90 degrees
- moved R7 45.2 mm to (29.2, 26.7), turned to 90 degrees
- moved R1 44.9 mm to (3.81, 72.4), turned to 180 degrees
- moved C1 35.6 mm to (17.8, 12.7)
- moved C5 35.6 mm to (17.8, 20.3)
- moved J1 31.8 mm to (10.2, 53.3)
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Connections:
- net GND: no longer S1.3, S1.4
- net RESET: no longer S1.1, S1.2
Routing:
- net +3.3V: track 0.00 -> 151.3 mm, vias 0 -> 1
- net ARD0_FLASH: track 0.00 -> 110.3 mm, vias 0 -> 2
- net TXD: track 0.00 -> 84.9 mm
- net ENABLE: track 0.00 -> 82.3 mm, vias 0 -> 2
- net RXD: track 0.00 -> 78.3 mm
- net ARD05: track 0.00 -> 62.3 mm, vias 0 -> 1
- net RESET: track 0.00 -> 61.8 mm, vias 0 -> 3
- net GND: track 0.00 -> 58.4 mm, vias 0 -> 2
- net ARD04: track 0.00 -> 50.0 mm, vias 0 -> 1
- net ARD02: track 0.00 -> 43.2 mm, vias 0 -> 1
- net ARD12: track 0.00 -> 39.5 mm, vias 0 -> 1
- net ARD13: track 0.00 -> 34.1 mm, vias 0 -> 1
- net CTRL-: track 0.00 -> 30.7 mm
- net DOOR+: track 0.00 -> 17.8 mm, vias 0 -> 1
- net N$1: track 0.00 -> 15.2 mm
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- added copper zone on layer 16, net GND
Other:
- board size 100 x 80 mm -> 34 x 78.7 mm

Commit message: Mostly final board design
Parts:
- added A_LED, S_LED: (no value), adafruit:LED5MM
- added R8: 250, resistor:M3216
- C1, C2: value (none) -> 100pF
- CTRL_OUT: value ILD2 -> OPTOCOUPLER
- D1: value BAS40 -> Schottky Diodes; device diode:SOT23 -> diode:SMB
- D2, D3: value BAS40 -> (none); device diode:SOT23 -> diode:SMB
- IC2: value REG1117 -> AMS1117-3.3V
- R5: value 10K -> 250
- moved R5 25.7 mm to (25.4, 47.0)
- moved C3 6.35 mm to (17.8, 43.2)
- moved C5 6.35 mm to (17.8, 14.0)
- moved C1 4.02 mm to (21.6, 14.0)
- moved C2 3.81 mm to (21.6, 20.3)
- moved C6 3.81 mm to (17.8, 20.3)
- moved D1 2.54 mm to (19.1, 8.89)
- moved CTRL_OUT 1.80 mm to (25.4, 40.6)
- moved IC2 1.27 mm to (22.9, 53.3)
- moved JP1 1.27 mm to (20.3, 3.81)
- moved IC1 1.27 mm to (3.81, 67.3)
- moved R2 0.63 mm to (8.26, 67.3)
- turned C7 to 270 degrees
- turned R6 to 270 degrees
- renumbered DOOR_CLOSED_SENSOR to DOOR_CLOSED, DOOR_UP_SENSOR to DOOR_OPEN
Connections:
- new net N$4: R5.1, S_LED.K
- new net N$5: A_LED.K, R8.1
- new net N$6: R5.2
- new net N$7: S_LED.A
- new net N$8: A_LED.A
- net +3.3V: no longer R5.1
- net ARD02: no longer R5.2
- net ARD0_FLASH: now also D3.A; no longer D3.1
- net GND: now also R8.2
- net N$1: now also D2.A, D3.C; no longer D2.1, D3.3
- net N$2: now also D2.C; no longer D2.3
- net RXD: now also D1.A; no longer D1.1
- net RXD_5V: now also D1.C; no longer D1.3
Routing:
- net ARD0_FLASH: track 110.3 -> 66.4 mm, vias 2 -> 3
- net RESET: track 61.8 -> 92.0 mm, vias 3 -> 2
- net +3.3V: track 151.3 -> 132.9 mm, vias 1 -> 0
- net N$5: track 0.00 -> 14.0 mm
- net TXD: track 84.9 -> 72.3 mm, vias 0 -> 1
- net ENABLE: track 82.3 -> 73.0 mm
- net ARD04: track 50.0 -> 58.2 mm
- net N$4: track 0.00 -> 8.17 mm
- net ARD02: track 43.2 -> 37.1 mm, vias 1 -> 0
- net ARD12: track 39.5 -> 33.9 mm, vias 1 -> 0
- net GND: track 58.4 -> 63.3 mm
- net ARD05: track 62.3 -> 66.8 mm
- net RXD: track 78.3 -> 82.6 mm
- net DOOR+: track 17.8 -> 13.8 mm, vias 1 -> 0
- net N$2: track 2.71 -> 6.16 mm
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
Commit message: Closer to final board design
Parts:
- IC2: value AMS1117-3.3V -> 3.3V REG
Connections:
- removed net N$6: R5.2
- removed net N$7: S_LED.A
- removed net N$8: A_LED.A
- new net ARD16: A_LED.A, U$1.GPIO16
- net ARD14: now also S_LED.A
- net ARD15: now also R5.2
Routing:
- net ARD16: track 0.00 -> 60.4 mm, vias 0 -> 1
- net +3.3V: track 132.9 -> 188.7 mm, vias 0 -> 1
- net ARD14: track 0.00 -> 31.3 mm
- net ARD15: track 0.00 -> 16.2 mm
- net RESET: track 92.0 -> 76.0 mm, vias 2 -> 0
- net ARD05: track 66.8 -> 81.2 mm
- net RXD: track 82.6 -> 93.1 mm, vias 0 -> 2
- net GND: track 63.3 -> 56.8 mm, vias 2 -> 3
- net ARD12: track 33.9 -> 29.9 mm
- net TXD: track 72.3 -> 75.6 mm, vias 1 -> 0
- net ARD13: track 33.1 -> 36.3 mm, vias 2 -> 0
- net CTRL-: track 29.1 -> 31.1 mm
- net ARD04: track 58.2 -> 59.8 mm, vias 1 -> 0
- net ARD02: track 37.1 -> 35.9 mm, vias 0 -> 1
- net LIGHTS+: track 15.4 -> 14.4 mm, vias 1 -> 0
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Other:
- board text added: "DTR GRN"
- board text added: "ESP8266 Garage Door Monitor April 2016 KJA"
- board text added: "FTDI Connector"
- board text added: "GND BLK"
