File: hardware/boards/gdo_v7/gdo_v7.sch (EAGLE design)
At the start: 30 parts, among them IC2 3.3V REG, J1 PJ-036AH-SMT-TR, Q1 BSS84, Q2 BSS138, Q3 BSS138, Q4 IRLML2502, U1 PC817XI

Commit message: Initial commit of the v7 board designs
Parts:
- C1, C2, C4, C5: device resistor:C-EUC1206 -> resistor:C-USC0805
- Q4: value IRLML2502 -> 2502
Changed lines of the file:
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@@
 <part name="GND3" library="supply1" deviceset="GND" device=""/>
 <part name="GND4" library="supply1" deviceset="GND" device=""/>
-<part name="C1" library="resistor" deviceset="C-EU" device="C1206" value="100pF"/>
-<part name="C2" library="resistor" deviceset="C-EU" device="C1206" value="100pF"/>
+<part name="C1" library="resistor" library_urn="urn:adsk.eagle:library:348" deviceset="C-US" device="C0805" package3d_urn="urn:adsk.eagle:package:26137/1" value="100pF"/>
+<part name="C2" library="resistor" library_urn="urn:adsk.eagle:library:348" deviceset="C-US" device="C0805" package3d_urn="urn:adsk.eagle:package:26137/1" value="100pF"/>
 <part name="GND7" library="supply1" deviceset="GND" device=""/>
 <part name="JP1" library="adafruit" deviceset="PINHD-1X6" device=""/>
@@
 <part name="C8" library="SparkFun-Capacitors" deviceset="10UF-TANT" device="" value="22uF"/>
 <part name="C9" library="SparkFun-Capacitors" deviceset="10UF-TANT" device="" value="22uF"/>
-<part name="C4" library="resistor" deviceset="C-EU" device="C1206" value="100nF"/>
+<part name="C4" library="resistor" library_urn="urn:adsk.eagle:library:348" deviceset="C-US" device="C0805" package3d_urn="urn:adsk.eagle:package:26137/1" value="100nF"/>
 <part name="Q1" library="transistor-small-signal" deviceset="BSS84" device=""/>
 <part name="Q2" library="Ava" deviceset="BSS138" device=""/>
@@
 <part name="R2" library="resistor" library_urn="urn:adsk.eagle:library:348" deviceset="R-US_" device="R0805" package3d_urn="urn:adsk.eagle:package:26059/1" value="100k"/>
 <part name="R3" library="resistor" library_urn="urn:adsk.eagle:library:348" deviceset="R-US_" device="R0805" package3d_urn="urn:adsk.eagle:package:26059/1" value="100k"/>
-<part name="C5" library="resistor" deviceset="C-EU" device="C1206" value="100nF"/>
+<part name="C5" library="resistor" library_urn="urn:adsk.eagle:library:348" deviceset="C-US" device="C0805" package3d_urn="urn:adsk.eagle:package:26137/1" value="100nF"/>
 <part name="R4" library="resistor" library_urn="urn:adsk.eagle:library:348" deviceset="R-US_" device="R0805" package3d_urn="urn:adsk.eagle:package:26059/1" value="100k"/>
 <part name="GND8" library="supply1" deviceset="GND" device=""/>
@@
 <part name="P+1" library="supply1" deviceset="+5V" device=""/>
 <part name="GND1" library="supply1" deviceset="GND" device=""/>
-<part name="Q4" library="bss138_10" deviceset="BSS138" device="" value="IRLML2502"/>
+<part name="Q4" library="bss138_10" deviceset="BSS138" device="" value="2502"/>
 <part name="R7" library="resistor" library_urn="urn:adsk.eagle:library:348" deviceset="R-US_" device="R0805" package3d_urn="urn:adsk.eagle:package:26059/1" value="4.7kΩ"/>
 <part name="R8" library="resistor" library_urn="urn:adsk.eagle:library:348" deviceset="R-US_" device="R0805" package3d_urn="urn:adsk.eagle:package:26059/1" value="10k"/>
@@
 </instance>
 <instance part="C4" gate="G$1" x="17.272" y="72.136" smashed="yes">
-<attribute name="NAME" x="18.796" y="72.517" size="1.016" layer="95" align="center"/>
+<attribute name="NAME" x="19.05" y="73.025" size="1.016" layer="95" align="center"/>
 <attribute name="VALUE" x="19.812" y="69.215" size="1.016" layer="96" align="center"/>
 </instance>
